File: RpiOnOff.sch (EAGLE design)
At the start: 22 parts, among them CON1 CONNECTOR-1X2[2.54MM], CON2 CONNECTOR-1X2[2.54MM], Q1 BSS84, Q2 BSS123

Commit message: I think the main change was fixing a transistor footprint.
This is the version that was sent for production to Seeed Studios.
Parts:
- C1: device rcl:C-EUC0805 -> Erland's Library:C-EUC0603
- Q1: value BSS84 -> MOSFET-P-TOSHIBA-SSM3J338R; device transistor-small-signal:BSS84 -> Erland's Library:MOSFET-P-TOSHIBA-SSM3J338R
- Q2: value BSS123 -> MOSFET-N-SSM3K36MFV; device transistor-small-signal:BSS123 -> Erland's Library:MOSFET-N-SSM3K36MFV
- R1, R2, R4, R5, R6, R7: device rcl:R-EU_R0603 -> Erland's Library:R-EU_R0603
- R3: device rcl:R-EU_R0805 -> Erland's Library:R-EU_R0603
Connections:
- net +5V: now also Q1.S; no longer Q1.D
- net VDD: now also Q1.D; no longer Q1.S
Other:
- moved on the sheet: CON1, JP1, X2-1, X2-2
